File: kicad_files/key.kicad_pcb (KiCad board)
At the start: 2 copper layers, 10 parts, among them IC1 ATTINY85-P, P1 USB_A, SW1 SW_PUSH

Commit message: New PCB design
Parts:
- removed D1, D2: D, Diodes_SMD:D_SMA_Standard
- removed the D3 at (106.0, 64.8)
- removed the P1 at (98.9, 52.7)
- added 1.5k1: R, Resistors_SMD:R_1206, F.Cu at (164.2, 48.5)
- added 1.5k1: R, Resistors_SMD:R_1206, F.Cu at (196.0, 48.5)
- added 1.5k1: R, Resistors_SMD:R_1206, F.Cu at (255.7, 47.2)
- added 1.5k1: R, Resistors_SMD:R_1206, F.Cu at (223.9, 47.2)
- added 1.5k1: R, Resistors_SMD:R_1206, F.Cu at (109.6, 48.5)
- added 1.5k1: R, Resistors_SMD:R_1206, F.Cu at (141.4, 48.5)
- added 1.5k1: R, Resistors_SMD:R_1206, F.Cu at (81.7, 49.8)
- added 1.5k2: R, Resistors_SMD:R_1206, F.Cu at (166.6, 48.1)
- added 1.5k2: R, Resistors_SMD:R_1206, F.Cu at (198.4, 48.1)
- added 1.5k2: R, Resistors_SMD:R_1206, F.Cu at (258.1, 46.9)
- added 1.5k2: R, Resistors_SMD:R_1206, F.Cu at (226.3, 46.9)
- added 1.5k2: R, Resistors_SMD:R_1206, F.Cu at (112.0, 48.1)
- added 1.5k2: R, Resistors_SMD:R_1206, F.Cu at (143.8, 48.1)
- added 1.5k2: R, Resistors_SMD:R_1206, F.Cu at (84.1, 49.4)
- added D3: LED, LEDs:LED_0402, F.Cu at (168.3, 53.3)
- added D3: LED, LEDs:LED_0402, F.Cu at (200.0, 53.3)
- added D3: LED, LEDs:LED_0402, F.Cu at (259.7, 52.1)
- added D3: LED, LEDs:LED_0402, F.Cu at (228.0, 52.1)
- added D3: LED, LEDs:LED_0402, F.Cu at (113.7, 53.3)
- added D3: LED, LEDs:LED_0402, F.Cu at (145.4, 53.3)
- added D3: LED, LEDs:LED_0402, F.Cu at (85.7, 54.6)
- added D3: LED, LEDs:LED_0402, F.Cu at (54.0, 54.6)
- added IC1: ATTINY85-P, SOIC127P600X175-8N:SOIC127P600X175-8N, F.Cu at (162.8, 56.1)
- added IC1: ATTINY85-P, SOIC127P600X175-8N:SOIC127P600X175-8N, F.Cu at (194.6, 56.1)
- added IC1: ATTINY85-P, SOIC127P600X175-8N:SOIC127P600X175-8N, F.Cu at (254.3, 54.9)
- added IC1: ATTINY85-P, SOIC127P600X175-8N:SOIC127P600X175-8N, F.Cu at (222.5, 54.9)
- added IC1: ATTINY85-P, SOIC127P600X175-8N:SOIC127P600X175-8N, F.Cu at (108.2, 56.1)
- added IC1: ATTINY85-P, SOIC127P600X175-8N:SOIC127P600X175-8N, F.Cu at (140.0, 56.1)
- added IC1: ATTINY85-P, SOIC127P600X175-8N:SOIC127P600X175-8N, F.Cu at (80.3, 57.4)
- added P1: USB_A, kicad_files:usb-PCB, F.Cu at (165.1, 36.8)
- added P1: USB_A, kicad_files:usb-PCB, F.Cu at (196.8, 36.8)
- added P1: USB_A, kicad_files:usb-PCB, F.Cu at (256.5, 35.6)
- added P1: USB_A, kicad_files:usb-PCB, F.Cu at (224.8, 35.6)
- added P1: USB_A, kicad_files:usb-PCB, F.Cu at (110.5, 36.8)
- added P1: USB_A, kicad_files:usb-PCB, F.Cu at (142.2, 36.8)
- added P1: USB_A, kicad_files:usb-PCB, F.Cu at (82.5, 38.1)
- added P1: USB_A, kicad_files:usb-PCB, F.Cu at (50.8, 38.1)
- added R1: R, Resistors_SMD:R_1206, F.Cu at (161.9, 48.1)
- added R1: R, Resistors_SMD:R_1206, F.Cu at (193.7, 48.1)
- added R1: R, Resistors_SMD:R_1206, F.Cu at (253.4, 46.9)
- added R1: R, Resistors_SMD:R_1206, F.Cu at (221.6, 46.9)
- added R1: R, Resistors_SMD:R_1206, F.Cu at (107.3, 48.1)
- added R1: R, Resistors_SMD:R_1206, F.Cu at (139.1, 48.1)
- added R1: R, Resistors_SMD:R_1206, F.Cu at (79.4, 49.4)
- added R2: R, Resistors_SMD:R_1206, F.Cu at (167.3, 58.3)
- added R2: R, Resistors_SMD:R_1206, F.Cu at (199.0, 58.3)
- added R2: R, Resistors_SMD:R_1206, F.Cu at (258.7, 57.0)
- added R2: R, Resistors_SMD:R_1206, F.Cu at (226.9, 57.0)
- added R2: R, Resistors_SMD:R_1206, F.Cu at (112.6, 58.3)
- added R2: R, Resistors_SMD:R_1206, F.Cu at (144.4, 58.3)
- added R2: R, Resistors_SMD:R_1206, F.Cu at (84.7, 59.6)
- added SW1: SW_PUSH, Buttons_Switches_SMD:SW_SPST_FSMSM, F.Cu at (167.1, 67.3)
- added SW1: SW_PUSH, Buttons_Switches_SMD:SW_SPST_FSMSM, F.Cu at (198.9, 67.3)
- added SW1: SW_PUSH, Buttons_Switches_SMD:SW_SPST_FSMSM, F.Cu at (258.6, 66.0)
- added SW1: SW_PUSH, Buttons_Switches_SMD:SW_SPST_FSMSM, F.Cu at (226.8, 66.0)
- added SW1: SW_PUSH, Buttons_Switches_SMD:SW_SPST_FSMSM, F.Cu at (112.5, 67.3)
- added SW1: SW_PUSH, Buttons_Switches_SMD:SW_SPST_FSMSM, F.Cu at (144.3, 67.3)
- added SW1: SW_PUSH, Buttons_Switches_SMD:SW_SPST_FSMSM, F.Cu at (84.6, 68.6)
- moved IC1 55.9 mm to (48.5, 57.4), turned to 90 degrees
- moved SW1 53.1 mm to (52.8, 68.6)
- moved R1 51.9 mm to (47.6, 49.4), turned to 90 degrees
- moved 1.5k2 51.3 mm to (52.3, 49.4), turned to 270 degrees
- moved R2 50.4 mm to (53.0, 59.6), turned to 270 degrees
- moved 1.5k1 50.3 mm to (49.9, 49.8)
Connections:
- 1.5k1 pad 1: D- -> D+
- 1.5k2 pad 1: D+ -> D-
- IC1 pad 1: Net-(IC1-Pad1) -> (no net)
- IC1 pad 2: Net-(IC1-Pad2) -> B
- IC1 pad 7: B -> (no net)
- R1 pad 2: D- -> D+
Routing:
- net GND: track 0.19 -> 94.0 mm
- net +5V: track 22.7 -> 103.7 mm
- net Net-(1.5k2-Pad2): track 8.45 -> 78.1 mm
- net B: track 10.2 -> 63.7 mm
- net Net-(IC1-Pad3): track 6.66 -> 47.9 mm
- net D+: track 23.0 -> 62.8 mm
- net D-: track 8.87 -> 42.4 mm
- net Net-(D3-Pad2): track 2.56 -> 31.0 mm
- net Net-(1.5k1-Pad2): track 7.82 -> 28.2 mm
Other:
- net class Default: trace_width 0.3048 -> 0.4
