File: kicad_files/key.sch (KiCad schematic (older format))
At the start: 10 parts, among them IC1 ATTINY85-P, P1 USB_A, SW1 SW_PUSH

Commit message: New PCB design
Parts:
- removed D1, D2: D, Diodes_SMD:D_SMA_Standard, symbol D
- P1: footprint Connectors:USB_A -> kicad_files:usb-PCB
Connections:
- net B: now also IC1.2 (PB3(XTAL1/CLKI/OC1B/ADC3/PCINT3)); no longer IC1.7 (PB2(SCK/USCK/SCL/T0/INT0/ADC1/PCINT2))
- net D+: now also 1.5k1.1, R1.2; no longer 1.5k2.1
- net D-: now also 1.5k2.1; no longer 1.5k1.1, R1.2
Other:
- moved on the sheet: 1.5k1, 1.5k2, D3, R1, R2
Changed lines of the file:
@@
-$EndComp
-$Comp
-L D D1
-U 1 1 58D80332
-P 2500 4950
-F 0 "D1" H 2500 5050 50  0000 C CNN
-F 1 "D" H 2500 4850 50  0000 C CNN
-F 2 "Diodes_SMD:D_SMA_Standard" H 2500 4950 50  0001 C CNN
-F 3 "" H 2500 4950 50  0000 C CNN
-	1    2500 4950
-	0    1    1    0
 $EndComp
 $Comp
 L R 1.5k1
 U 1 1 58D80594
-P 3700 3500
-F 0 "1.5k1" V 3780 3500 50  0000 C CNN
-F 1 "R" V 3700 3500 50  0000 C CNN
-F 2 "Resistors_SMD:R_1206" V 3630 3500 50  0001 C CNN
-F 3 "" H 3700 3500 50  0000 C CNN
-	1    3700 3500
+P 3650 3750
+F 0 "1.5k1" V 3730 3750 50  0000 C CNN
+F 1 "R" V 3650 3750 50  0000 C CNN
+F 2 "Resistors_SMD:R_1206" V 3580 3750 50  0001 C CNN
+F 3 "" H 3650 3750 50  0000 C CNN
+	1    3650 3750
 	0    -1   -1   0
 $EndComp
@@
 L R R2
 U 1 1 58D80E01
-P 4000 3950
-F 0 "R2" V 4080 3950 50  0000 C CNN
-F 1 "R" V 4000 3950 50  0000 C CNN
-F 2 "Resistors_SMD:R_1206" V 3930 3950 50  0001 C CNN
-F 3 "" H 4000 3950 50  0000 C CNN
-	1    4000 3950
+P 3950 4200
+F 0 "R2" V 4030 4200 50  0000 C CNN
+F 1 "R" V 3950 4200 50  0000 C CNN
+F 2 "Resistors_SMD:R_1206" V 3880 4200 50  0001 C CNN
+F 3 "" H 3950 4200 50  0000 C CNN
+	1    3950 4200
 	0    -1   -1   0
 $EndComp
@@
 L R R1
 U 1 1 58D8152B
-P 2500 4200
-F 0 "R1" V 2580 4200 50  0000 C CNN
-F 1 "R" V 2500 4200 50  0000 C CNN
-F 2 "Resistors_SMD:R_1206" V 2430 4200 50  0001 C CNN
-F 3 "" H 2500 4200 50  0000 C CNN
-	1    2500 4200
-	1    0    0    -1
-$EndComp
-$Comp
-L D D2
-U 1 1 58D81ACC
-P 3000 4950
-F 0 "D2" H 3000 5050 50  0000 C CNN
-F 1 "D" H 3000 4850 50  0000 C CNN
-F 2 "Diodes_SMD:D_SMA_Standard" H 3000 4950 50  0001 C CNN
-F 3 "" H 3000 4950 50  0000 C CNN
-	1    3000 4950
-	0    1    1    0
+P 2450 4450
+F 0 "R1" V 2530 4450 50  0000 C CNN
+F 1 "R" V 2450 4450 50  0000 C CNN
+F 2 "Resistors_SMD:R_1206" V 2380 4450 50  0001 C CNN
+F 3 "" H 2450 4450 50  0000 C CNN
+	1    2450 4450
+	1    0    0    -1
 $EndComp
 $Comp
 L GND #PWR03
-U 1 1 58D81B31
-P 2500 5350
-F 0 "#PWR03" H 2500 5100 50  0001 C CNN
-F 1 "GND" H 2500 5200 50  0000 C CNN
-F 2 "" H 2500 5350 50  0000 C CNN
-F 3 "" H 2500 5350 50  0000 C CNN
-	1    2500 5350
-	1    0    0    -1
-$EndComp
-$Comp
-L GND #PWR04
 U 1 1 58D81B63
 P 2700 2900
-F 0 "#PWR04" H 2700 2650 50  0001 C CNN
+F 0 "#PWR03" H 2700 2650 50  0001 C CNN
 F 1 "GND" H 2700 2750 50  0000 C CNN
 F 2 "" H 2700 2900 50  0000 C CNN
@@
 $EndComp
 $Comp
-L GND #PWR05
-U 1 1 58D81C93
-P 3000 5350
-F 0 "#PWR05" H 3000 5100 50  0001 C CNN
-F 1 "GND" H 3000 5200 50  0000 C CNN
-F 2 "" H 3000 5350 50  0000 C CNN
-F 3 "" H 3000 5350 50  0000 C CNN
-	1    3000 5350
-	1    0    0    -1
-$EndComp
-$Comp
-L GND #PWR06
+L GND #PWR04
 U 1 1 58D81D88
 P 2000 2750
-F 0 "#PWR06" H 2000 2500 50  0001 C CNN
+F 0 "#PWR04" H 2000 2500 50  0001 C CNN
 F 1 "GND" H 2000 2600 50  0000 C CNN
 F 2 "" H 2000 2750 50  0000 C CNN
@@
 $EndComp
 $Comp
-L +5V #PWR07
+L +5V #PWR05
 U 1 1 58D81DC9
 P 1700 2750
-F 0 "#PWR07" H 1700 2600 50  0001 C CNN
+F 0 "#PWR05" H 1700 2600 50  0001 C CNN
 F 1 "+5V" H 1700 2890 50  0000 C CNN
 F 2 "" H 1700 2750 50  0000 C CNN
@@
 $EndComp
 $Comp
-L +5V #PWR08
+L +5V #PWR06
 U 1 1 58D81E9E
-P 2500 3900
-F 0 "#PWR08" H 2500 3750 50  0001 C CNN
-F 1 "+5V" H 2500 4040 50  0000 C CNN
-F 2 "" H 2500 3900 50  0000 C CNN
-F 3 "" H 2500 3900 50  0000 C CNN
-	1    2500 3900
-	1    0    0    -1
-$EndComp
-Text GLabel 2150 4650 0    60   Input ~ 0
+P 2450 4150
+F 0 "#PWR06" H 2450 4000 50  0001 C CNN
+F 1 "+5V" H 2450 4290 50  0000 C CNN
+F 2 "" H 2450 4150 50  0000 C CNN
+F 3 "" H 2450 4150 50  0000 C CNN
+	1    2450 4150
+	1    0    0    -1
+$EndComp
+Text GLabel 3300 4950 2    60   Input ~ 0
 D-
-Text GLabel 3350 4700 2    60   Input ~ 0
+Text GLabel 2100 4900 0    60   Input ~ 0
 D+
 Text GLabel 1700 3350 3    60   Input ~ 0
@@
 L R 1.5k2
 U 1 1 58D821C9
-P 3700 3600
-F 0 "1.5k2" V 3780 3600 50  0000 C CNN
-F 1 "R" V 3700 3600 50  0000 C CNN
-F 2 "Resistors_SMD:R_1206" V 3630 3600 50  0001 C CNN
-F 3 "" H 3700 3600 50  0000 C CNN
-	1    3700 3600
+P 3650 3850
+F 0 "1.5k2" V 3730 3850 50  0000 C CNN
+F 1 "R" V 3650 3850 50  0000 C CNN
+F 2 "Resistors_SMD:R_1206" V 3580 3850 50  0001 C CNN
+F 3 "" H 3650 3850 50  0000 C CNN
+	1    3650 3850
 	0    -1   -1   0
 $EndComp
 NoConn ~ 4150 2500
 $Comp
-L GND #PWR09
+L GND #PWR07
 U 1 1 58E47062
-P 3300 4150
-F 0 "#PWR09" H 3300 3900 50  0001 C CNN
-F 1 "GND" H 3300 4000 50  0000 C CNN
-F 2 "" H 3300 4150 50  0000 C CNN
-F 3 "" H 3300 4150 50  0000 C CNN
-	1    3300 4150
+P 3250 4400
+F 0 "#PWR07" H 3250 4150 50  0001 C CNN
+F 1 "GND" H 3250 4250 50  0000 C CNN
+F 2 "" H 3250 4400 50  0000 C CNN
+F 3 "" H 3250 4400 50  0000 C CNN
+	1    3250 4400
 	1    0    0    -1
 $EndComp
 Text GLabel 4200 2900 2    60   Input ~ 0
 B
-Text GLabel 4150 3400 0    60   Input ~ 0
-B
 $Comp
 L LED D3
 U 1 1 58EA4021
-P 3550 3950
-F 0 "D3" H 3550 4050 50  0000 C CNN
-F 1 "LED" H 3550 3850 50  0000 C CNN
-F 2 "LEDs:LED_0402" H 3550 3950 50  0001 C CNN
-F 3 "" H 3550 3950 50  0000 C CNN
-	1    3550 3950
+P 3500 4200
+F 0 "D3" H 3500 4300 50  0000 C CNN
+F 1 "LED" H 3500 4100 50  0000 C CNN
+F 2 "LEDs:LED_0402" H 3500 4200 50  0001 C CNN
+F 3 "" H 3500 4200 50  0000 C CNN
+	1    3500 4200
 	1    0    0    -1
 $EndComp
@@
 F 0 "P1" H 2100 1950 50  0000 C CNN
 F 1 "USB_A" H 1850 2350 50  0000 C CNN
-F 2 "Connectors:USB_A" V 1850 2050 50  0001 C CNN
+F 2 "kicad_files:usb-PCB" V 1850 2050 50  0001 C CNN
 F 3 "" V 1850 2050 50  0000 C CNN
 	1    1900 2150
@@
 	1700 2750 1700 2450
 Wire Wire Line
-	2500 5100 2500 5350
-Wire Wire Line
-	2500 4350 2500 4800
-Connection ~ 2500 4650
-Wire Wire Line
-	2500 3900 2500 4050
-Wire Wire Line
-	2150 4650 2700 4650
+	2450 4600 2450 4900
+Connection ~ 2450 4900
+Wire Wire Line
+	2450 4150 2450 4300
+Wire Wire Line
+	2100 4900 2650 4900
 Wire Wire Line
 	1800 2450 1800 3150
@@
 	2000 3150 2000 3350
 Wire Wire Line
-	3550 3600 3000 3600
-Wire Wire Line
-	3000 3600 3000 4800
-Wire Wire Line
-	3350 4700 3000 4700
-Connection ~ 3000 4700
-Wire Wire Line
-	3550 3500 2700 3500
-Wire Wire Line
-	2700 3500 2700 4650
+	3500 3850 2950 3850
+Wire Wire Line
+	2950 3850 2950 4950
+Wire Wire Line
+	2950 4950 3300 4950
+Connection ~ 2950 4950
+Wire Wire Line
+	3500 3750 2650 3750
+Wire Wire Line
+	2650 3750 2650 4900
 Wire Wire Line
 	4200 2900 3900 2900
@@
 	7100 3700 7100 3850
 Wire Wire Line
-	3000 5100 3000 5350
-Wire Wire Line
-	3700 3950 3850 3950
+	3650 4200 3800 4200
 Wire Wire Line
 	2700 2900 3300 2900
 Wire Wire Line
-	3300 3950 3400 3950
-Wire Wire Line
-	3300 3950 3300 4150
-Wire Wire Line
-	4150 3400 4300 3400
-Wire Wire Line
-	3850 3500 3850 3200
+	3250 4200 3350 4200
+Wire Wire Line
+	3250 4200 3250 4400
+Text GLabel 4100 3750 3    60   Input ~ 0
+B
+Wire Wire Line
+	3800 3750 3850 3750
+Wire Wire Line
+	3850 3750 3850 3200
 Wire Wire Line
 	3850 3200 4300 3200
 Wire Wire Line
-	3850 3600 3950 3600
-Wire Wire Line
-	3950 3600 3950 3300
+	3800 3850 3950 3850
+Wire Wire Line
+	3950 3850 3950 3300
 Wire Wire Line
 	3950 3300 4300 3300
 Wire Wire Line
-	4300 3600 4150 3600
-Wire Wire Line
-	4150 3600 4150 3950
+	4100 4200 4250 4200
+Wire Wire Line
+	4250 4200 4250 3600
+Wire Wire Line
+	4250 3600 4300 3600
+Wire Wire Line
+	4300 3500 4100 3500
+Wire Wire Line
+	4100 3500 4100 3750
 $EndSCHEMATC
